File: masterpod_pcb_kicad/Vibro_Band.kicad_pcb (KiCad board)
At the start: 2 copper layers, 9 parts, among them U1 ULN2003A, U2 MPU-6050, U3 XIAO-ESP32-C3-SMD

Commit message: finished pcb?
Parts:
- removed BAT1, MTR1, MTR2, MTR3, MTR4: Conn_01x02_Pin, TestPoint:TestPoint_2Pads_Pitch2.54mm_Drill0.8mm
- removed C1: C_US, Capacitor_THT:CP_Radial_D6.3mm_P2.50mm
- removed U2: MPU-6050, GY-521:MODULE_GY-521
- added J1: Conn_01x04_Socket, Connector_PinSocket_2.54mm:PinSocket_1x04_P2.54mm_Horizontal, F.Cu at (153.6, 120.3)
- added J2: Conn_01x06_Socket, Connector_PinSocket_2.54mm:PinSocket_1x06_P2.54mm_Horizontal, F.Cu at (136.5, 107.4)
- added J3: Conn_01x08_Socket, Connector_PinSocket_2.54mm:PinSocket_1x08_P2.54mm_Horizontal, F.Cu at (136.4, 82.6)
- added SW1: SW_SPDT, Button_Switch_THT:SW_Slide_SPDT_Angled_CK_OS102011MA1Q, F.Cu at (161.6, 103.8)
- moved U3 48.6 mm to (143.5, 94.5)
- moved U1 47.1 mm to (150.0, 101.9)
Connections:
- U1 pad 9: /ESP_BAT+ -> /3.3V
- U3 pad 12: Net-(SW1A-B) -> /3.3V
- U3 pad 17: CHIP_EN -> /CHIP_EN
- U3 pad 21: /ESP_BAT+ -> /BAT+
- U3 pad 22: /ESP_BAT- -> /BAT-
Routing:
- net /GND: track 0.00 -> 121.0 mm, vias 0 -> 1
- net /3.3V: track 0.00 -> 57.3 mm, vias 0 -> 2
- net /MTR4+: track 0.00 -> 56.9 mm, vias 0 -> 2
- net /MTR3+: track 0.00 -> 54.4 mm, vias 0 -> 2
- net /BAT-: track 0.00 -> 40.1 mm, vias 0 -> 2
- net /MTR2+: track 0.00 -> 37.2 mm, vias 0 -> 2
- net /MTR1+: track 0.00 -> 34.5 mm
- net /BAT+: track 0.00 -> 32.3 mm, vias 0 -> 2
- net /CHIP_EN: track 0.00 -> 31.5 mm, vias 0 -> 1
- net /TRAN1: track 0.00 -> 28.7 mm, vias 0 -> 2
- net /TRAN2: track 0.00 -> 28.0 mm, vias 0 -> 2
- net /TRAN3: track 0.00 -> 27.4 mm
- net /TRAN4: track 0.00 -> 22.9 mm, vias 0 -> 2
- net /SDA: track 0.00 -> 13.0 mm
- net /SCL: track 0.00 -> 12.0 mm
- added copper zone on B.Cu, net /GND
- added copper zone on F.Cu, net /GND
Other:
- board outline added: 31 x 50 mm

Commit message: updates to kicad
Parts:
- J1: moved to B.Cu
- U1: footprint Package_SO:SOIC-16_3.9x9.9mm_P1.27mm -> Package_DIP:DIP-16_W7.62mm
- moved J1 50.4 mm to (198.6, 97.7)
- moved J2 49.9 mm to (185.4, 97.7)
- moved J3 49.6 mm to (185.4, 75.1)
- moved SW1 45.8 mm to (206.0, 115.0)
- moved U3 44.7 mm to (188.2, 94.2)
- moved U1 38.6 mm to (188.4, 97.4)
Connections:
- J1 pad 1: /MTR3+ -> /BAT+
- J1 pad 2: /GND -> /MTR3-
- J1 pad 3: /MTR4+ -> /BAT+
- J1 pad 4: /GND -> /MTR4-
- J2 pad 3: /MTR1+ -> /BAT+
- J2 pad 4: /GND -> /MTR1-
- J2 pad 5: /MTR2+ -> /BAT+
- J2 pad 6: /GND -> /MTR2-
- U1 pad 13: /MTR4+ -> /MTR4-
- U1 pad 14: /MTR3+ -> /MTR3-
- U1 pad 15: /MTR2+ -> /MTR2-
- U1 pad 16: /MTR1+ -> /MTR1-
Routing:
- net /MTR4+: track 56.9 -> 0.00 mm, vias 2 -> 0
- net /MTR3+: track 54.4 -> 0.00 mm, vias 2 -> 0
- net /MTR2+: track 37.2 -> 0.00 mm, vias 2 -> 0
- net /GND: track 121.0 -> 84.3 mm
- net /MTR1+: track 34.5 -> 0.00 mm
- net /CHIP_EN: track 31.5 -> 54.5 mm
- net /BAT+: track 32.3 -> 51.9 mm, vias 2 -> 1
- net /BAT-: track 40.1 -> 22.5 mm, vias 2 -> 1
- net /MTR2-: track 0.00 -> 15.8 mm
- net /MTR1-: track 0.00 -> 13.9 mm
- net /TRAN4: track 22.9 -> 33.8 mm, vias 2 -> 1
- net /SDA: track 13.0 -> 3.99 mm
- net /SCL: track 12.0 -> 3.99 mm
- net /TRAN3: track 27.4 -> 32.3 mm, vias 0 -> 1
- net /MTR3-: track 0.00 -> 3.56 mm
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- removed copper zone on B.Cu, net /GND
- removed copper zone on F.Cu, net /GND
Other:
- board size 31 x 50 mm -> 31 x 46.5 mm
- board text added: "Texas Robotics Medical Robotics & Haptics Designed By: Connor M. & Kishore K."
