File: masterpod_pcb_kicad/Vibro_Band.kicad_sch (KiCad schematic)
At the start: 11 parts, among them SW1 SW_DPST_x2, U1 ULN2003A, U2 MPU-6050, U3 XIAO-ESP32-C3-SMD

Commit message: finished pcb?
Parts:
- removed BAT1, MTR1, MTR2, MTR3, MTR4: Conn_01x02_Pin, TestPoint:TestPoint_2Pads_Pitch2.54mm_Drill0.8mm, symbol Connector:Conn_01x02_Pin
- removed C1: C_US, Capacitor_THT:CP_Radial_D6.3mm_P2.50mm, symbol Device:C_US
- removed SW1: SW_DPST_x2, SW_Slide_SPDT_SS12D07, symbol Switch:SW_DPST_x2
- removed U2: MPU-6050, GY-521:MODULE_GY-521, symbol Sensor_Motion:MPU-6050
- added J1: Conn_01x04_Socket, Connector_PinSocket_2.54mm:PinSocket_1x04_P2.54mm_Horizontal, symbol Connector:Conn_01x04_Socket
- added J2: Conn_01x06_Socket, Connector_PinSocket_2.54mm:PinSocket_1x06_P2.54mm_Horizontal, symbol Connector:Conn_01x06_Socket
- added J3: Conn_01x08_Socket, Connector_PinSocket_2.54mm:PinSocket_1x08_P2.54mm_Horizontal, symbol Connector:Conn_01x08_Socket
- added SW1: SW_SPDT, Button_Switch_THT:SW_Slide_SPDT_Angled_CK_OS102011MA1Q, symbol Switch:SW_SPDT
Connections:
- net GND: now also J1.2 (Pin_2), J1.4 (Pin_4), J2.4 (Pin_4), J2.6 (Pin_6), J3.7 (Pin_7), SW1.1 (A)
- net MTR1+: now also J2.3 (Pin_3)
- net MTR2+: now also J2.5 (Pin_5)
- net MTR3+: now also J1.1 (Pin_1)
- net MTR4+: now also J1.3 (Pin_3)
- net SCL: now also J3.6 (Pin_6)
- net SDA: now also J3.5 (Pin_5)
- net 3.3V: now reaches U3.12 (3V3)
- net 3.3V: now also U1.9 (COM), J3.8 (Pin_8)
- net CHIP_EN: now reaches U3.26 (CHIP_EN)
- net CHIP_EN: now also SW1.2 (B)
- net ESP_BAT+ renamed BAT+
- net BAT+: now also J2.1 (Pin_1); no longer U1.9 (COM)
- net ESP_BAT- renamed BAT-
- net BAT-: now also J2.2 (Pin_2)
Other:
- note removed: "Battery Pad J5"

Commit message: updates to kicad
Parts:
- U1: footprint Package_SO:SOIC-16_3.9x9.9mm_P1.27mm -> Package_DIP:DIP-16_W7.62mm
Connections:
- net BAT+: now also J1.1 (Pin_1), J1.3 (Pin_3), J2.3 (Pin_3), J2.5 (Pin_5)
- net GND: no longer J1.2 (Pin_2), J1.4 (Pin_4), J2.4 (Pin_4), J2.6 (Pin_6)
- net MTR1+ renamed MTR1-
- net MTR1-: now also J2.4 (Pin_4); no longer J2.3 (Pin_3)
- net MTR2+ renamed MTR2-
- net MTR2-: now also J2.6 (Pin_6); no longer J2.5 (Pin_5)
- net MTR3+ renamed MTR3-
- net MTR3-: now also J1.2 (Pin_2); no longer J1.1 (Pin_1)
- net MTR4+ renamed MTR4-
- net MTR4-: now also J1.4 (Pin_4); no longer J1.3 (Pin_3)
Other:
- note added: "This switch powers on the board, if CHIP_EN is floating then chip enabled"
- note removed: "This switch powers on the board, if CHIP_EN is high then chip enabled"
