File: masterpod_pcb_kicad/Vibro_Band.kicad_sch (KiCad schematic)
At the start: 7 parts, among them J1 Conn_01x04_Socket, J2 Conn_01x06_Socket, J3 Conn_01x08_Socket, SW1 SW_SPDT, U1 ULN2003A, U3 XIAO-ESP32-C3-SMD

Commit message: updates to readme and cleanup of unsed functions
Co-authored-by: Copilot <copilot@github.com>
Parts:
- removed LIPO_Battery1: 3.7V, symbol Device:Battery
Other:
- company: (none) -> Medical Robotics & Haptics FRI, HERO Lab, Texas Robotics, Connor M & Kishore K
- title: (none) -> TACTUS | Vibrotactile Band for Learning Large Motor Skills
- moved on the sheet: J1, J2, J3, SW1, U1
